File: hardware/icarus/icarus.sch (KiCad schematic (older format))
At the start: 43 parts, among them J1 USB_B_Micro, J2 SWJ-DP, J3 PWR, J4 PWM, J5 COMMS, J6 GPIO, SW1 RST, SW2 BOOT, U1 STM32F302C8Tx, U2 AMS1117-3.3, U3 MPU-6050, Y1 12MHz

Commit message: Resolves #4. Increased resistor values for LEDs
Parts:
- R2, R6, R7: value 100 -> 200; LCSC C17408 -> C17540
Changed lines of the file:
@@
 P 3600 1750
 F 0 "R2" H 3670 1796 50  0000 L CNN
-F 1 "100" H 3670 1705 50  0000 L CNN
+F 1 "200" H 3670 1705 50  0000 L CNN
 F 2 "Resistor_SMD:R_0805_2012Metric" V 3530 1750 50  0001 C CNN
 F 3 "~" H 3600 1750 50  0001 C CNN
-F 4 "C17408" H 3600 1750 50  0001 C CNN "LCSC"
+F 4 "C17540" H 3600 1750 50  0001 C CNN "LCSC"
 	1    3600 1750
 	1    0    0    -1
@@
 P 12250 1700
 F 0 "R6" H 12320 1746 50  0000 L CNN
-F 1 "100" H 12320 1655 50  0000 L CNN
+F 1 "200" H 12320 1655 50  0000 L CNN
 F 2 "Resistor_SMD:R_0805_2012Metric" V 12180 1700 50  0001 C CNN
 F 3 "~" H 12250 1700 50  0001 C CNN
-F 4 "C17408" H 12250 1700 50  0001 C CNN "LCSC"
+F 4 "C17540" H 12250 1700 50  0001 C CNN "LCSC"
 	1    12250 1700
 	1    0    0    -1
@@
 P 12750 1700
 F 0 "R7" H 12820 1746 50  0000 L CNN
-F 1 "100" H 12820 1655 50  0000 L CNN
+F 1 "200" H 12820 1655 50  0000 L CNN
 F 2 "Resistor_SMD:R_0805_2012Metric" V 12680 1700 50  0001 C CNN
 F 3 "~" H 12750 1700 50  0001 C CNN
-F 4 "C17408" H 12750 1700 50  0001 C CNN "LCSC"
+F 4 "C17540" H 12750 1700 50  0001 C CNN "LCSC"
 	1    12750 1700
 	1    0    0    -1
