File: hardware/icarus/icarus.kicad_sch (KiCad schematic)
At the start: 43 parts, among them J1 USB_B_Micro, J2 SWJ-DP, J3 PWR, J4 PWM, J5 COMMS, J6 GPIO, SW1 RST, SW2 BOOT, U1 STM32F302C8Tx, U2 AMS1117-3.3, U3 MPU-6050, Y1 12MHz

Commit message: Resolves #3, #13. Use 5 pin header for SWD, Use SOT-89 package for regulator.
Parts:
- removed J2: SWJ-DP, Connector_PinHeader_1.27mm:PinHeader_2x05_P1.27mm_Vertical_SMD, symbol Connector:Conn_ARM_JTAG_SWD_10
- removed J3: PWR, Connector_PinSocket_2.54mm:PinSocket_1x06_P2.54mm_Vertical, symbol Connector_Generic:Conn_01x06
- removed J4: PWM, Connector_PinSocket_2.54mm:PinSocket_1x06_P2.54mm_Vertical, symbol Connector_Generic:Conn_01x06
- removed J5: COMMS, Connector_PinSocket_2.54mm:PinSocket_1x06_P2.54mm_Vertical, symbol Connector_Generic:Conn_01x06
- removed J6: GPIO, Connector_PinSocket_2.54mm:PinSocket_1x08_P2.54mm_Vertical, symbol Connector_Generic:Conn_01x08
- added J?: SWD, symbol Connector_Generic:Conn_01x05
- added U?: ICARUS, icarus:icarus-shield, symbol icarus:ICARUS
- U2: footprint Package_TO_SOT_SMD:SOT-223-3_TabPin2 -> Package_TO_SOT_SMD:SOT-89-3; LCSC C6186 -> C880752
Connections:
- net gpio4 is gone; now on net gpio2: U1.22 (PB11)
- net gpio5 is gone; now on net gpio3: U1.25 (PB12)
- net +3V3: now also J?.1 (Pin_1), U?.7 (3V3)
- net GND: now also J?.5 (Pin_5), U?.2 (GND), U?.4 (GND), U?.6 (GND), U?.8 (GND)
- net VBUS: now also U?.5 (5V)
- net VDC: now also U?.1 (VDC), U?.3 (VDC)
- net gpio1: now also U1.21 (PB10), U?.15 (GPIO1); no longer U1.45 (PB8)
- net gpio2: now also U?.16 (GPIO2); no longer U1.46 (PB9)
- net gpio3: now also U?.17 (GPIO3); no longer U1.21 (PB10)
- net miso: now also U?.22 (MISO)
- net mosi: now also U?.20 (MOSI)
- net nreset: now also J?.4 (Pin_4)
- net pwm1: now also U?.9 (PWM1)
- net pwm2: now also U?.10 (PWM2)
- net pwm3: now also U?.11 (PWM3)
- net pwm4: now also U?.12 (PWM4)
- net pwm5: now also U?.13 (PWM5)
- net pwm6: now also U?.14 (PWM6)
- net sck: now also U?.18 (SCK)
- net scl: now also U?.27 (SCL)
- net sda: now also U?.28 (SDA)
- net swclk: now also J?.2 (Pin_2)
- net swdio: now also J?.3 (Pin_3)
- net usart1_rx: now also U?.23 (RX0)
- net usart1_tx: now also U?.24 (TX0)
- net usart2_rx: now also U?.25 (RX1)
- net usart2_tx: now also U?.26 (TX1)
- new net can_rx: U1.45 (PB8), U?.19 (CAN_RX)
- new net can_tx: U1.46 (PB9), U?.21 (CAN_TX)
Other:
- note added: "Shield"
- note removed: "Breakout"

Commit message: Resolves #5. Smaller push buttons for BOOT and RST
Parts:
- SW1, SW2: footprint Button_Switch_SMD:SW_Push_1P1T_NO_6x6mm_H9.5mm -> tactile_switches:TS-1088-AR02016; LCSC C127509 -> C720477
Changed lines of the file:
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@@
     (property "Reference" "SW2" (id 0) (at 171.45 72.771 0))
     (property "Value" "BOOT" (id 1) (at 171.45 75.0824 0))
-    (property "Footprint" "Button_Switch_SMD:SW_Push_1P1T_NO_6x6mm_H9.5mm" (id 2) (at 171.45 74.93 0)
+    (property "Footprint" "tactile_switches:TS-1088-AR02016" (id 2) (at 171.45 74.93 0)
       (effects (font (size 1.27 1.27)) hide)
     )
@@
       (effects (font (size 1.27 1.27)) hide)
     )
-    (property "LCSC" "C127509" (id 4) (at 171.45 80.01 0)
+    (property "LCSC" "C720477" (id 4) (at 171.45 80.01 0)
       (effects (font (size 1.27 1.27)) hide)
     )
@@
       (effects (font (size 1.27 1.27)) (justify left))
     )
-    (property "Footprint" "Button_Switch_SMD:SW_Push_1P1T_NO_6x6mm_H9.5mm" (id 2) (at 144.78 83.82 0)
+    (property "Footprint" "tactile_switches:TS-1088-AR02016" (id 2) (at 144.78 83.82 0)
       (effects (font (size 1.27 1.27)) hide)
     )
@@
       (effects (font (size 1.27 1.27)) hide)
     )
-    (property "LCSC" "C127509" (id 4) (at 139.7 83.82 90)
+    (property "LCSC" "C720477" (id 4) (at 139.7 83.82 90)
       (effects (font (size 1.27 1.27)) hide)
     )
@@
     )
     (path "/00000000-0000-0000-0000-000061786c85"
-      (reference "SW1") (unit 1) (value "RST") (footprint "Button_Switch_SMD:SW_Push_1P1T_NO_6x6mm_H9.5mm")
+      (reference "SW1") (unit 1) (value "RST") (footprint "tactile_switches:TS-1088-AR02016")
     )
     (path "/00000000-0000-0000-0000-0000617444a3"
-      (reference "SW2") (unit 1) (value "BOOT") (footprint "Button_Switch_SMD:SW_Push_1P1T_NO_6x6mm_H9.5mm")
+      (reference "SW2") (unit 1) (value "BOOT") (footprint "tactile_switches:TS-1088-AR02016")
     )
     (path "/00000000-0000-0000-0000-000061b20520"

Commit message: Resolves #1. Micro USB footprint selection
Parts:
- J1: footprint Connector_USB:USB_Micro-B_Amphenol_10103594-0001LF_Horizontal -> Connector_USB:USB_Micro-B_Molex_47346-0001; LCSC C132563 -> C132560
Changed lines of the file:
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@@
     (property "Reference" "J1" (id 0) (at 20.4978 23.6982 0))
     (property "Value" "USB_B_Micro" (id 1) (at 20.4978 26.0096 0))
-    (property "Footprint" "Connector_USB:USB_Micro-B_Amphenol_10103594-0001LF_Horizontal" (id 2) (at 22.86 36.83 0)
+    (property "Footprint" "Connector_USB:USB_Micro-B_Molex_47346-0001" (id 2) (at 22.86 36.83 0)
       (effects (font (size 1.27 1.27)) hide)
     )
@@
       (effects (font (size 1.27 1.27)) hide)
     )
-    (property "LCSC" "C132563" (id 4) (at 19.05 35.56 0)
+    (property "LCSC" "C132560" (id 4) (at 19.05 35.56 0)
       (effects (font (size 1.27 1.27)) hide)
     )
@@
     )
     (path "/00000000-0000-0000-0000-0000615e41e1"
-      (reference "J1") (unit 1) (value "USB_B_Micro") (footprint "Connector_USB:USB_Micro-B_Amphenol_10103594-0001LF_Horizontal")
+      (reference "J1") (unit 1) (value "USB_B_Micro") (footprint "Connector_USB:USB_Micro-B_Molex_47346-0001")
     )
     (path "/c65b3c44-ecd3-4a11-89a8-fa4dca44bae9"

Commit message: Resolves #6, #17, #18. Resize and routing. Added barometer.
Parts:
- removed TP?: SWCLK, symbol Connector:TestPoint
- removed TP?: SWDIO, symbol Connector:TestPoint
- removed TP?: RX1, symbol Connector:TestPoint
- removed TP?: TX1, symbol Connector:TestPoint
- removed TP?: RX2, symbol Connector:TestPoint
- removed TP?: TX2, symbol Connector:TestPoint
- removed TP?: SCL, symbol Connector:TestPoint
- removed TP?: SDA, symbol Connector:TestPoint
- removed TP?: RST, symbol Connector:TestPoint
- added C12, C2: 100nF, Capacitor_SMD:C_0805_2012Metric, symbol Device:C
- added U4: BMP388, sensors:BMP388, symbol sensors:BMP388
- J2: renamed from J?; footprint (none) -> custom-breakout:SWD-bcu
- TP1, TP2, TP3: renamed from TP?; footprint (none) -> TestPoint:TestPoint_Pad_1.0x1.0mm
- gave numbers to parts that had none: 1
Connections:
- net +3V3: now also C12.1, C2.1, U4.1 (VDDIO), U4.10 (VDD), U4.5 (SDO), U4.6 (CSB)
- net GND: now also C12.2, C2.2, U4.3 (GND), U4.8 (GND), U4.9 (GND)
- net scl: now also U4.2 (SCK)
- net sda: now also U4.4 (SDI)
- no-connect marks 3 -> 4
Other:
- note added: "Altitude Sensing"
- note added: "I2C Addresses: $68"
- note added: "I2C Addresses: $77"
- moved on the sheet: TP1, TP2, TP3

Commit message: Added LCSC to BMP on schematic
Parts:
- U4: LCSC (none) -> C779278
Changed lines of the file:
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@@
+      (effects (font (size 1.27 1.27)) hide)
+    )
+    (property "LCSC" "C779278" (id 4) (at 252.73 208.28 0)
       (effects (font (size 1.27 1.27)) hide)
     )

Commit message: kibot ci
Parts:
- Y1: LCSC C669076 -> C669076
Changed lines of the file:
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@@
       (effects (font (size 1.27 1.27)) hide)
     )
-    (property "Datasheet" "~" (id 3) (at 22.86 36.83 0)
+    (property "Datasheet" "https://datasheet.lcsc.com/lcsc/1811141734_MOLEX-473460001_C132560.pdf" (id 3) (at 22.86 36.83 0)
       (effects (font (size 1.27 1.27)) hide)
     )
@@
       (effects (font (size 1.27 1.27)) hide)
     )
-    (property "Datasheet" "~" (id 3) (at 111.76 30.48 0)
+    (property "Datasheet" "https://datasheet.lcsc.com/lcsc/1810261822_Samsung-Electro-Mechanics-CL21A475KAQNNNE_C1779.pdf" (id 3) (at 111.76 30.48 0)
       (effects (font (size 1.27 1.27)) hide)
     )
@@
       (effects (font (size 1.27 1.27)) hide)
     )
-    (property "Datasheet" "~" (id 3) (at 153.67 30.48 0)
+    (property "Datasheet" "https://datasheet.lcsc.com/lcsc/1810191216_Samsung-Electro-Mechanics-CL21B104KCFNNNE_C28233.pdf" (id 3) (at 153.67 30.48 0)
       (effects (font (size 1.27 1.27)) hide)
     )
@@
       (effects (font (size 1.27 1.27)) hide)
     )
-    (property "Datasheet" "~" (id 3) (at 162.56 30.48 0)
+    (property "Datasheet" "https://datasheet.lcsc.com/lcsc/1810191216_Samsung-Electro-Mechanics-CL21B104KCFNNNE_C28233.pdf" (id 3) (at 162.56 30.48 0)
       (effects (font (size 1.27 1.27)) hide)
     )
@@
       (effects (font (size 1.27 1.27)) hide)
     )
-    (property "Datasheet" "~" (id 3) (at 171.45 30.48 0)
+    (property "Datasheet" "https://datasheet.lcsc.com/lcsc/1810191216_Samsung-Electro-Mechanics-CL21B104KCFNNNE_C28233.pdf" (id 3) (at 171.45 30.48 0)
       (effects (font (size 1.27 1.27)) hide)
     )
@@
       (effects (font (size 1.27 1.27)) hide)
     )
-    (property "Datasheet" "~" (id 3) (at 128.27 83.82 0)
+    (property "Datasheet" "https://datasheet.lcsc.com/lcsc/1810191216_Samsung-Electro-Mechanics-CL21B104KCFNNNE_C28233.pdf" (id 3) (at 128.27 83.82 0)
       (effects (font (size 1.27 1.27)) hide)
     )
@@
       (effects (font (size 1.27 1.27)) hide)
     )
-    (property "Datasheet" "~" (id 3) (at 135.89 170.18 0)
-      (effects (font (size 1.27 1.27)) hide)
-    )
-    (property "LCSC" " C669076 " (id 4) (at 135.89 170.18 0)
+    (property "Datasheet" "https://datasheet.lcsc.com/lcsc/2103291236_Yangxing-Tech-OT201612MJBA4SL_C669076.pdf" (id 3) (at 135.89 170.18 0)
+      (effects (font (size 1.27 1.27)) hide)
+    )
+    (property "LCSC" "C669076" (id 4) (at 135.89 170.18 0)
       (effects (font (size 1.27 1.27)) hide)
     )
@@
       (effects (font (size 1.27 1.27)) hide)
     )
-    (property "Datasheet" "~" (id 3) (at 91.44 31.75 0)
+    (property "Datasheet" "https://datasheet.lcsc.com/lcsc/1912111437_Yongyu-Photoelectric-SZYY0805G_C434432.pdf" (id 3) (at 91.44 31.75 0)
       (effects (font (size 1.27 1.27)) hide)
     )
@@
       (effects (font (size 1.27 1.27)) hide)
     )
-    (property "Datasheet" "~" (id 3) (at 91.44 44.45 0)
+    (property "Datasheet" "https://datasheet.lcsc.com/lcsc/2110251830_UNI-ROYAL-Uniroyal-Elec-0805W8F2000T5E_C17540.pdf" (id 3) (at 91.44 44.45 0)
       (effects (font (size 1.27 1.27)) hide)
     )
@@
       (effects (font (size 1.27 1.27)) hide)
     )
-    (property "Datasheet" "https://store.invensense.com/datasheets/invensense/MPU-6050_DataSheet_V3%204.pdf" (id 3) (at 166.37 226.06 0)
+    (property "Datasheet" "https://invensense.tdk.com/wp-content/uploads/2015/02/MPU-6000-Datasheet1.pdf" (id 3) (at 166.37 226.06 0)
       (effects (font (size 1.27 1.27)) hide)
     )
@@
       (effects (font (size 1.27 1.27)) hide)
     )
-    (property "Datasheet" "~" (id 3) (at 160.02 85.09 0)
+    (property "Datasheet" "https://datasheet.lcsc.com/lcsc/2110251730_UNI-ROYAL-Uniroyal-Elec-0805W8F1002T5E_C17414.pdf" (id 3) (at 160.02 85.09 0)
       (effects (font (size 1.27 1.27)) hide)
     )
@@
       (effects (font (size 1.27 1.27)) hide)
     )
-    (property "Datasheet" "~" (id 3) (at 171.45 74.93 0)
+    (property "Datasheet" "https://datasheet.lcsc.com/lcsc/2008221234_XUNPU-TS-1088-AR02016_C720477.pdf" (id 3) (at 171.45 74.93 0)
       (effects (font (size 1.27 1.27)) hide)
     )
@@
       (effects (font (size 1.27 1.27)) hide)
     )
-    (property "Datasheet" "~" (id 3) (at 199.39 236.22 0)
+    (property "Datasheet" "https://datasheet.lcsc.com/lcsc/1810191215_Samsung-Electro-Mechanics-CL21C222JBFNNNE_C28260.pdf" (id 3) (at 199.39 236.22 0)
       (effects (font (size 1.27 1.27)) hide)
     )
@@
       (effects (font (size 1.27 1.27)) hide)
     )
-    (property "Datasheet" "~" (id 3) (at 186.69 236.22 0)
+    (property "Datasheet" "https://datasheet.lcsc.com/lcsc/1810191216_Samsung-Electro-Mechanics-CL21B104KCFNNNE_C28233.pdf" (id 3) (at 186.69 236.22 0)
       (effects (font (size 1.27 1.27)) hide)
     )
@@
       (effects (font (size 1.27 1.27)) hide)
     )
-    (property "Datasheet" "~" (id 3) (at 144.78 83.82 0)
+    (property "Datasheet" "https://datasheet.lcsc.com/lcsc/2008221234_XUNPU-TS-1088-AR02016_C720477.pdf" (id 3) (at 144.78 83.82 0)
       (effects (font (size 1.27 1.27)) hide)
     )
@@
       (effects (font (size 1.27 1.27)) hide)
     )
-    (property "Datasheet" "~" (id 3) (at 311.15 33.02 0)
+    (property "Datasheet" "https://datasheet.lcsc.com/lcsc/1912111437_Yongyu-Photoelectric-SZYY0805G_C434432.pdf" (id 3) (at 311.15 33.02 0)
       (effects (font (size 1.27 1.27)) hide)
     )
@@
       (effects (font (size 1.27 1.27)) hide)
     )
-    (property "Datasheet" "~" (id 3) (at 323.85 33.02 0)
+    (property "Datasheet" "https://datasheet.lcsc.com/lcsc/1912111437_Yongyu-Photoelectric-SZYY0805G_C434432.pdf" (id 3) (at 323.85 33.02 0)
       (effects (font (size 1.27 1.27)) hide)
     )
@@
       (effects (font (size 1.27 1.27)) hide)
     )
-    (property "Datasheet" "~" (id 3) (at 311.15 43.18 0)
+    (property "Datasheet" "https://datasheet.lcsc.com/lcsc/2110251830_UNI-ROYAL-Uniroyal-Elec-0805W8F2000T5E_C17540.pdf" (id 3) (at 311.15 43.18 0)
       (effects (font (size 1.27 1.27)) hide)
     )
@@
       (effects (font (size 1.27 1.27)) hide)
     )
-    (property "Datasheet" "~" (id 3) (at 323.85 43.18 0)
+    (property "Datasheet" "https://datasheet.lcsc.com/lcsc/2110251830_UNI-ROYAL-Uniroyal-Elec-0805W8F2000T5E_C17540.pdf" (id 3) (at 323.85 43.18 0)
       (effects (font (size 1.27 1.27)) hide)
     )
@@
       (effects (font (size 1.27 1.27)) hide)
     )
-    (property "Datasheet" "~" (id 3) (at 204.47 213.36 0)
+    (property "Datasheet" "https://datasheet.lcsc.com/lcsc/1811151136_Samsung-Electro-Mechanics-CL21B103KBANNNC_C1710.pdf" (id 3) (at 204.47 213.36 0)
       (effects (font (size 1.27 1.27)) hide)
     )
@@
       (effects (font (size 1.27 1.27)) hide)
     )
-    (property "Datasheet" "~" (id 3) (at 214.63 213.36 0)
+    (property "Datasheet" "https://datasheet.lcsc.com/lcsc/1810191216_Samsung-Electro-Mechanics-CL21B104KCFNNNE_C28233.pdf" (id 3) (at 214.63 213.36 0)
       (effects (font (size 1.27 1.27)) hide)
     )
@@
       (effects (font (size 1.27 1.27)) hide)
     )
-    (property "Datasheet" "~" (id 3) (at 74.93 35.56 0)
+    (property "Datasheet" "https://datasheet.lcsc.com/lcsc/1809281513_KEMET-T491A226K010AT_C116575.pdf" (id 3) (at 74.93 35.56 0)
       (effects (font (size 1.27 1.27)) hide)
     )
@@
       (effects (font (size 1.27 1.27)) hide)
     )
-    (property "Datasheet" "~" (id 3) (at 119.38 219.71 0)
+    (property "Datasheet" "https://datasheet.lcsc.com/lcsc/2110251730_UNI-ROYAL-Uniroyal-Elec-0805W8F1002T5E_C17414.pdf" (id 3) (at 119.38 219.71 0)
       (effects (font (size 1.27 1.27)) hide)
     )
@@
       (effects (font (size 1.27 1.27)) hide)
     )
-    (property "Datasheet" "~" (id 3) (at 119.38 228.6 0)
+    (property "Datasheet" "https://datasheet.lcsc.com/lcsc/2110251730_UNI-ROYAL-Uniroyal-Elec-0805W8F1002T5E_C17414.pdf" (id 3) (at 119.38 228.6 0)
       (effects (font (size 1.27 1.27)) hide)
     )
@@
       (effects (font (size 1.27 1.27)) hide)
     )
-    (property "Datasheet" "~" (id 3) (at 354.33 184.15 0)
+    (property "Datasheet" "" (id 3) (at 354.33 184.15 0)
       (effects (font (size 1.27 1.27)) hide)
     )
@@
       (effects (font (size 1.27 1.27)) hide)
     )
-    (property "Datasheet" "~" (id 3) (at 354.33 189.23 0)
+    (property "Datasheet" "" (id 3) (at 354.33 189.23 0)
       (effects (font (size 1.27 1.27)) hide)
     )
@@
       (effects (font (size 1.27 1.27)) hide)
     )
-    (property "Datasheet" "~" (id 3) (at 354.33 194.31 0)
+    (property "Datasheet" "" (id 3) (at 354.33 194.31 0)
       (effects (font (size 1.27 1.27)) hide)
     )
@@
       (effects (font (size 1.27 1.27)) hide)
     )
-    (property "Datasheet" "~" (id 3) (at 270.51 212.09 0)
+    (property "Datasheet" "https://datasheet.lcsc.com/lcsc/1810191216_Samsung-Electro-Mechanics-CL21B104KCFNNNE_C28233.pdf" (id 3) (at 270.51 212.09 0)
       (effects (font (size 1.27 1.27)) hide)
     )
@@
       (effects (font (size 1.27 1.27)) hide)
     )
-    (property "Datasheet" "~" (id 3) (at 167.64 124.46 0)
+    (property "Datasheet" "" (id 3) (at 167.64 124.46 0)
       (effects (font (size 1.27 1.27)) hide)
     )
@@
       (effects (font (size 1.27 1.27)) hide)
     )
-    (property "Datasheet" "" (id 3) (at 259.08 207.01 0)
+    (property "Datasheet" "https://datasheet.lcsc.com/lcsc/2110191430_Bosch-Sensortec-BMP388_C779278.pdf" (id 3) (at 259.08 207.01 0)
       (effects (font (size 1.27 1.27)) hide)
     )
@@
       (effects (font (size 1.27 1.27)) hide)
     )
-    (property "Datasheet" "~" (id 3) (at 283.21 212.09 0)
-      (effects (font (size 1.27 1.27)) hide)
-    )
+    (property "Datasheet" "https://datasheet.lcsc.com/lcsc/1810191216_Samsung-Electro-Mechanics-CL21B104KCFNNNE_C28233.pdf" (id 3) (at 283.21 212.09 0)
+      (effects (font (size 1.27 1.27)) hide)
+    )

Commit message: Rev C
Parts:
- removed C3: 4.7uF, Capacitor_SMD:C_0805_2012Metric, symbol Device:C
- removed C5, C7: 100nF, Capacitor_SMD:C_0805_2012Metric, symbol Device:C
- removed D2: STAT1, LED_SMD:LED_0805_2012Metric, symbol Device:LED
- removed J1: USB_B_Micro, Connector_USB:USB_Micro-B_Molex_47346-0001, symbol Connector:USB_B_Micro
- removed J2: SWD, custom-breakout:SWD-bcu, symbol Connector_Generic:Conn_01x05
- removed R4: 10k, Resistor_SMD:R_0805_2012Metric, symbol Device:R
- removed U1: STM32F302C8Tx, Package_QFP:LQFP-48_7x7mm_P0.5mm, symbol MCU_ST_STM32F3:STM32F302C8Tx
- removed U5: ICARUS, icarus:icarus-shield, symbol icarus:ICARUS
- removed Y1: 12MHz, Crystal:Crystal_SMD_2016-4Pin_2.0x1.6mm, symbol Device:Crystal_GND24
- added C10: 100nF, Capacitor_SMD:C_0402_1005Metric, symbol Device:C
- added D1: B5819W, Diode_SMD:D_SOD-123, symbol Device:D_Schottky
- added D4: STAT, LED_SMD:LED_WS2812B_PLCC4_5.0x5.0mm_P3.2mm, symbol LED:WS2812B
- added D5: CHR, LED_SMD:LED_0805_2012Metric, symbol Device:LED
- added J1: BAT, Connector_PinHeader_2.54mm:PinHeader_1x02_P2.54mm_Vertical, symbol Connector_Generic:Conn_01x02
- added M1: RTR1, Connector_PinHeader_2.54mm:PinHeader_1x02_P2.54mm_Vertical, symbol Motor:Motor_DC
- added M2: RTR2, Connector_PinHeader_2.54mm:PinHeader_1x02_P2.54mm_Vertical, symbol Motor:Motor_DC
- added M3: RTR3, Connector_PinHeader_2.54mm:PinHeader_1x02_P2.54mm_Vertical, symbol Motor:Motor_DC
- added M4: RTR4, Connector_PinHeader_2.54mm:PinHeader_1x02_P2.54mm_Vertical, symbol Motor:Motor_DC
- added P1: USB_C_Plug_USB2.0, USB-C-Connectors:TYPE-C-31-M-04, symbol Connector:USB_C_Plug_USB2.0
- added Q1: DMG2305, Package_TO_SOT_SMD:SOT-23, symbol Device:Q_PMOS_GSD
- added Q2: 2N7002, Package_TO_SOT_SMD:SOT-23, symbol Transistor_FET:2N7002
- added R1, R9: 100k, Resistor_SMD:R_0402_1005Metric, symbol Device:R
- added R10: 1k, Resistor_SMD:R_0402_1005Metric, symbol Device:R
- added R11, R12, R13, R2: 10k, Resistor_SMD:R_0402_1005Metric, symbol Device:R
- added R8: 4.7k, Resistor_SMD:R_0402_1005Metric, symbol Device:R
- added TP4: GND, TestPoint:TestPoint_Pad_1.0x1.0mm, symbol Connector:TestPoint
- added U2, U3: DRV8837, Package_SON:WSON-8-1EP_2x2mm_P0.5mm_EP0.9x1.6mm, symbol Driver_Motor:DRV8837
- added U5: MCP73831-2-OT, Package_TO_SOT_SMD:SOT-23-5, symbol Battery_Management:MCP73831-2-OT
- added U7: ESP32-C3-MINI-1, Espressif:ESP32-C3-MINI-1, symbol Espressif:ESP32-C3-MINI-1
- C2: renamed from C8; footprint Capacitor_SMD:C_0805_2012Metric -> Capacitor_SMD:C_0402_1005Metric; LCSC C28233 -> C307331
- C3: renamed from C9; footprint Capacitor_SMD:C_0805_2012Metric -> Capacitor_SMD:C_0402_1005Metric; LCSC C28260 -> C1531
- C4: renamed from C10; footprint Capacitor_SMD:C_0805_2012Metric -> Capacitor_SMD:C_0402_1005Metric; LCSC C1710 -> C15195
- C5: renamed from C11; footprint Capacitor_SMD:C_0805_2012Metric -> Capacitor_SMD:C_0402_1005Metric; LCSC C28233 -> C307331
- C6: value 100nF -> 4.7uF; footprint Capacitor_SMD:C_0805_2012Metric -> Capacitor_SMD:C_0402_1005Metric; LCSC C28233 -> C23733
- C7: renamed from C2; footprint Capacitor_SMD:C_0805_2012Metric -> Capacitor_SMD:C_0402_1005Metric; LCSC C28233 -> C307331
- C8: renamed from C12; footprint Capacitor_SMD:C_0805_2012Metric -> Capacitor_SMD:C_0402_1005Metric; LCSC C28233 -> C307331
- C9: renamed from C4; footprint Capacitor_SMD:C_0805_2012Metric -> Capacitor_SMD:C_0402_1005Metric; LCSC C28233 -> C307331
- D2: renamed from D1; value PWR -> 5V
- D3: value STAT2 -> 3V3
- R3: footprint Resistor_SMD:R_0805_2012Metric -> Resistor_SMD:R_0402_1005Metric; LCSC C17414 -> C25744
- R4: renamed from R2; value 200 -> 1k; footprint Resistor_SMD:R_0805_2012Metric -> Resistor_SMD:R_0402_1005Metric; LCSC C17540 -> C25543
- R5: value 10k -> 560; footprint Resistor_SMD:R_0805_2012Metric -> Resistor_SMD:R_0402_1005Metric; LCSC C17414 -> C25172
- R6: value 200 -> 6.8k; footprint Resistor_SMD:R_0805_2012Metric -> Resistor_SMD:R_0402_1005Metric; LCSC C17540 -> C25917
- R7: value 200 -> 10k; footprint Resistor_SMD:R_0805_2012Metric -> Resistor_SMD:R_0402_1005Metric; LCSC C17540 -> C25744
- SW1: renamed from SW2; value BOOT -> USER
- TP1: value 3V3 -> VBUS
- TP2: value 5V -> BATT
- U1: renamed from U2; footprint Package_TO_SOT_SMD:SOT-89-3 -> Package_TO_SOT_SMD:SOT-223-3_TabPin2; LCSC C880752 -> C6186
- renumbered SW1 to SW2, U3 to U4, U4 to U6
Connections:
- net led2 is gone; now on net +3V3: D3.2 (A)
- net +3V3: now also R3.2, TP3.1, D4.1 (VDD), Q2.3 (D), R11.1, R12.1, R13.1, R2.2, U2.8 (VCC), U3.8 (VCC), U7.3 (3V3); no longer C6.1, D2.2 (A), R3.1, SW1.2, TP1.1
- net GND: now also SW1.1, C10.2, D4.3 (VSS), J1.2 (Pin_2), P1.A1 (GND), P1.A12 (GND), P1.B1 (GND), P1.B12 (GND), P1.S1 (SHIELD), R1.2, R8.2, R9.1, TP4.1, U2.4 (GND), U2.9 (GND), U3.4 (GND), U3.9 (GND), U5.2 (VSS), U7.1 (GND), U7.11 (GND), U7.14 (GND), U7.2 (GND), U7.36 (GND); no longer R6.2, TP3.1
- net VBUS: now also D2.2 (A), TP1.1, D1.2 (A), P1.A4 (VBUS), P1.A9 (VBUS), P1.B4 (VBUS), P1.B9 (VBUS), Q1.1 (G), R1.1, R10.2, U5.4 (VDD); no longer TP2.1, U1.3 (VI)
- net nreset: now also R11.2, U7.8 (EN/CHIP_PU)
- net scl: now also R3.1, U7.5 (GPIO2/ADC1_CH2)
- net sda: now also R2.1, U7.13 (GPIO1/ADC1_CH1/XTAL_32K_N); no longer R3.2
- net +BATT: now reaches R6.1
- net +BATT: now also C6.1, TP2.1, J1.1 (Pin_1), M1.1 (+), M2.1 (+), M3.1 (+), M4.1 (+), Q1.3 (D), U2.1 (VM), U3.1 (VM), U5.3 (VBAT)
- net at R7.1: now also R6.2, U7.6 (GPIO3/ADC1_CH3); no longer D3.1 (K)
- net boot0: no longer names the net of R5.1
- net boot0: now also D3.1 (K); no longer SW1.1
- net imu_int: no longer names the net of U4.12 (INT)
- new net: D1.1 (K), Q1.2 (S), U1.3 (VI)
- new net: M4.2 (-), U2.2 (OUT1)
- new net: M3.2 (-), U2.3 (OUT2)
- new net: M1.2 (-), U3.3 (OUT2)
- new net: D5.2 (A), R10.1
- new net: Q2.2 (S), R9.2, U7.12 (GPIO0/ADC1_CH0/XTAL_32K_P)
- new net: U3.7 (~{SLEEP}), U7.20 (GPIO6)
- new net: D4.4 (DIN), U7.31 (GPIO21/U0TXD)
- new net: R8.1, U5.5 (PROG)
- new net: M2.2 (-), U3.2 (OUT1)
- new net: D5.1 (K), Q2.1 (G), U5.1 (STAT)
- new net drv1_en: U2.7 (~{SLEEP}), U7.16 (GPIO10)
- new net rtrctl1: R13.2, U3.5 (IN2), U7.22 (GPIO8)
- new net rtrctl2: U3.6 (IN1), U7.21 (GPIO7)
- new net rtrctl3: U2.5 (IN2), U7.19 (GPIO5/ADC2_CH0)
- new net rtrctl4: U2.6 (IN1), U7.18 (GPIO4/ADC1_CH4)
- new net usb_dm: P1.A7 (D-), U7.26 (GPIO18/USB_D-)
- new net usb_dp: P1.A6 (D+), U7.27 (GPIO19/USB_D+)
- new net user_btn: C10.1, R12.2, SW1.2, U7.23 (GPIO9)
- no-connect marks 4 -> 8
Other:
- note added: "Battery Charge"
- note added: "Battery Sense"
- note added: "Boot Mode SPI Boot: GPIO2=1, GPIO8=x, GPIO9=1 Download: GPIO2=1, GPIO8=1, GPIO9=0"
- note added: "Charge Complete STAT=HIGH"
- note added: "Charge Current (mA) = 1000V / Rprog (k)"
- note added: "Independent Half-Bridge Configuration"
- note added: "MCU / RF"
- note added: "Max LiPo Voltage: 4.2V AREF: 2.5V"
- note added: "Motor Control"
- note added: "Power Supply"
- note added: "Reset / Boot Configuration Hold USER down, and press reset to enter Download mode"
- note added: "VBUS-BATT Isolation VBUS: Disconnected PMOS body diode is forward bias providing small leakage current. Resulting in Vgs < 0. Switching PMOS ON. VBUS: Connected Barrier diode is forward biased. Vgs=0. PMOS OFF."
- note removed: "Boot to system memory: BOOT0 - 1 nBOOT1 - 1 Boot to main flash memory: BOOT0 - 0 nBOOT1 - x"
- note removed: "Debugger Port"
- note removed: "Decoupling cap for each VDD pin on the MCU"
- note removed: "External Oscillator"
- note removed: "LED Indications"
- note removed: "MCU"
- note removed: "Power Filtering"
- note removed: "Reset / Boot Configuration"
- note removed: "Shield"
- note removed: "Single package oscillator. Output is a 12MHz clock signal (10ppm)"
- note removed: "Test Points"
- note removed: "USB / Power Input"
- moved on the sheet: C1, C2, C3, C4, C5, C7, C8, C9, D2, R4, SW1, SW2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
