File: hardware/icarus/icarus.kicad_sch (KiCad schematic)
At the start: 49 parts, among them J1 BAT, M1 RTR1, M2 RTR2, M3 RTR3, M4 RTR4, P1 USB_C_Plug_USB2.0, Q1 DMG2305, Q2 2N7002, SW1 USER, SW2 RST, U1 AMS1117-3.3, U2 DRV8837, U3 DRV8837, U4 MPU-6050, U5 MCP73831-2-OT, U6 BMP388, U7 ESP32-C3-MINI-1

Commit message: Rev D
Parts:
- removed C6: 4.7uF, Capacitor_SMD:C_0402_1005Metric, symbol Device:C
- removed D5: CHR, LED_SMD:LED_0805_2012Metric, symbol Device:LED
- removed M1: RTR1, Connector_PinHeader_2.54mm:PinHeader_1x02_P2.54mm_Vertical, symbol Motor:Motor_DC
- removed M2: RTR2, Connector_PinHeader_2.54mm:PinHeader_1x02_P2.54mm_Vertical, symbol Motor:Motor_DC
- removed M3: RTR3, Connector_PinHeader_2.54mm:PinHeader_1x02_P2.54mm_Vertical, symbol Motor:Motor_DC
- removed M4: RTR4, Connector_PinHeader_2.54mm:PinHeader_1x02_P2.54mm_Vertical, symbol Motor:Motor_DC
- removed Q2: 2N7002, Package_TO_SOT_SMD:SOT-23, symbol Transistor_FET:2N7002
- removed R10: 1k, Resistor_SMD:R_0402_1005Metric, symbol Device:R
- removed R7: 10k, Resistor_SMD:R_0402_1005Metric, symbol Device:R
- removed R8: 4.7k, Resistor_SMD:R_0402_1005Metric, symbol Device:R
- removed R9: 100k, Resistor_SMD:R_0402_1005Metric, symbol Device:R
- removed U2, U3: DRV8837, Package_SON:WSON-8-1EP_2x2mm_P0.5mm_EP0.9x1.6mm, symbol Driver_Motor:DRV8837
- removed U5: MCP73831-2-OT, Package_TO_SOT_SMD:SOT-23-5, symbol Battery_Management:MCP73831-2-OT
- added J2: IO, Connector_PinHeader_2.54mm:PinHeader_1x06_P2.54mm_Vertical, symbol Connector_Generic:Conn_01x06
- added J3: I2C_EX, Connector_PinHeader_2.54mm:PinHeader_1x02_P2.54mm_Vertical, symbol Connector_Generic:Conn_01x02
- added J4: UART, Connector_PinHeader_2.54mm:PinHeader_1x02_P2.54mm_Vertical, symbol Connector_Generic:Conn_01x02
- added U2: BMM150, Package_CSP:WLCSP-12_1.56x1.56mm_P0.4mm, symbol Sensor_Magnetic:BMM150
- R6: value 6.8k -> 10k; LCSC C25917 -> C25744
Connections:
- net +3V3: now also R6.1, U2.B2 (VDDIO), U2.E5 (VDD)
- net +BATT: no longer R6.1
- net GND: now also U2.A5 (CSB), U2.C1 (SDO), U2.C5 (GND), U2.E1 (GND), U2.E3 (GND)
- net scl: now also J3.2 (Pin_2), U2.A3 (SCK)
- net sda: now also J3.1 (Pin_1), U2.B4 (SDI)
- net at U7.12 (GPIO0/ADC1_CH0/XTAL_32K_P): now also D4.4 (DIN)
- net io5: now reaches U7.20 (GPIO6)
- net io5: now also J2.5 (Pin_5)
- net at U7.30 (GPIO20/U0RXD): now also J4.2 (Pin_2)
- net at U7.31 (GPIO21/U0TXD): now also J4.1 (Pin_1); no longer D4.4 (DIN)
- net at R6.2: now also U2.A1 (PS); no longer U7.6 (GPIO3/ADC1_CH3)
- net drv1_en renamed io2
- net io2: now also J2.2 (Pin_2)
- net rtrctl1: no longer names the net of R13.2, U7.22 (GPIO8)
- net rtrctl2 renamed io6
- net io6: now also J2.6 (Pin_6)
- net rtrctl3 renamed io4
- net io4: now also J2.4 (Pin_4)
- net rtrctl4 renamed io3
- net io3: now also J2.3 (Pin_3)
- new net io1: J2.1 (Pin_1), U7.6 (GPIO3/ADC1_CH3)
- no-connect marks 8 -> 10
Other:
- note added: "Accelerometer / Gyro"
- note added: "Barometer"
- note added: "I2C Address: $10"
- note added: "I2C Address: $68"
- note added: "I2C Address: $77"
- note added: "I2C Expansion Port"
- note added: "I2C Pullups"
- note added: "Magnetometer"
- note added: "Mode Select PS: 0=SPI, 1=I2C"
- note added: "PWM / DIO"
- note added: "STAT LED"
- note removed: "Altitude Sensing"
- note removed: "Battery Charge"
- note removed: "Battery Sense"
- note removed: "Charge Complete STAT=HIGH"
- note removed: "Charge Current (mA) = 1000V / Rprog (k)"
- note removed: "I2C Addresses: $68"
- note removed: "I2C Addresses: $77"
- note removed: "I2C Pullup"
- note removed: "Independent Half-Bridge Configuration"
- note removed: "Max LiPo Voltage: 4.2V AREF: 2.5V"
- note removed: "Motion Sensing"
- note removed: "Motor Control"
- moved on the sheet: C2, C3, C4, C5, C7, C8, D4, R13, R2, R3, TP1, TP2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
