File: hardware/icarus/icarus.kicad_sch (KiCad schematic)
At the start: 39 parts, among them J1 BAT, J2 IO, J3 I2C_EX, J4 UART, P1 USB_C_Plug_USB2.0, Q1 DMG2305, SW1 USER, SW2 RST, U1 AMS1117-3.3, U2 BMM150, U4 MPU-6050, U6 BMP388, U7 ESP32-C3-MINI-1

Commit message: Update actions
Parts:
- removed J4: UART, Connector_PinHeader_2.54mm:PinHeader_1x02_P2.54mm_Vertical, symbol Connector_Generic:Conn_01x02
- removed R13: 10k, Resistor_SMD:R_0402_1005Metric, symbol Device:R
- removed U7: ESP32-C3-MINI-1, Espressif:ESP32-C3-MINI-1, symbol Espressif:ESP32-C3-MINI-1
- added C11, C6: 20pF, Capacitor_SMD:C_0402_1005Metric, symbol Device:C
- added C12, C13: 2.2uF, Capacitor_SMD:C_0402_1005Metric, symbol Device:C
- added C14, C15, C17: 100nF, Capacitor_SMD:C_0402_1005Metric, symbol Device:C
- added C16: 4.7uF, Capacitor_SMD:C_0402_1005Metric, symbol Device:C
- added R7: 100, Resistor_SMD:R_0402_1005Metric, symbol Device:R
- added U3: STM32F405RGTx, Package_QFP:LQFP-64_10x10mm_P0.5mm, symbol MCU_ST_STM32F4:STM32F405RGTx
- added Y1: 12MHz, Crystal:Crystal_SMD_3225-4Pin_3.2x2.5mm, symbol Device:Crystal
- J3: value I2C_EX -> swd; footprint Connector_PinHeader_2.54mm:PinHeader_1x02_P2.54mm_Vertical -> Connector_PinHeader_1.00mm:PinHeader_1x02_P1.00mm_Vertical
- SW1: value USER -> BOOT
Connections:
- net +3V3: now also C10.1, C9.1, SW1.2, C14.1, C15.1, C16.1, C17.1, U3.13 (VDDA), U3.19 (VDD), U3.32 (VDD), U3.48 (VDD), U3.64 (VDD); no longer R12.1
- net GND: now also R12.2, C11.2, C12.2, C13.2, C14.2, C15.2, C16.2, C17.2, C6.2, U3.12 (VSSA), U3.18 (VSS), U3.28 (PB2), U3.63 (VSS); no longer SW1.1
- net nreset: now also U3.7 (NRST); no longer C9.1
- net scl: now also U3.58 (PB6); no longer J3.2 (Pin_2)
- net sda: now also U3.59 (PB7); no longer J3.1 (Pin_1)
- net usb_dm: now also U3.44 (PA11)
- net usb_dp: now also U3.45 (PA12)
- net at D4.4 (DIN): now also R7.2
- net io1 renamed pwm1
- net pwm1: now also U3.14 (PA0)
- net io2 renamed pwm2
- net pwm2: now also U3.15 (PA1)
- net io3 renamed pwm3
- net pwm3: now also U3.16 (PA2)
- net io4 renamed pwm4
- net pwm4: now also U3.17 (PA3)
- net io5 renamed usart_tx
- net usart_tx: now also U3.42 (PA9)
- net io6 renamed usart_rx
- net usart_rx: now also U3.43 (PA10)
- removed net user_btn: C10.1, R12.2, SW1.2
- new net: C12.1, U3.31 (VCAP_1)
- new net: C6.1, U3.5 (PH0), Y1.1
- new net: C11.1, U3.6 (PH1), Y1.2
- new net: C13.1, U3.47 (VCAP_2)
- new net boot0: R12.1, SW1.1, U3.60 (BOOT0)
- new net stat: R7.1, U3.26 (PB0)
- new net swclk: J3.2 (Pin_2), U3.49 (PA14)
- new net swdio: J3.1 (Pin_1), U3.46 (PA13)
- no-connect marks 10 -> 11
Other:
- note added: "Reset / Boot Configuration boot1=x,boot0=0 --> Main Flash boot1=0,boot0=1 --> System Memory"
- note removed: "Boot Mode SPI Boot: GPIO2=1, GPIO8=x, GPIO9=1 Download: GPIO2=1, GPIO8=1, GPIO9=0"
- note removed: "I2C Expansion Port"
- note removed: "MCU / RF"
- note removed: "PWM / DIO"
- note removed: "Reset / Boot Configuration Hold USER down, and press reset to enter Download mode"
- note removed: "STAT LED"
- moved on the sheet: C2, C3, C4, C5, C7, C8, D4, R11, R12, R2, R3, R6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

Commit message: add stm32 lcsc number
Parts:
- U3: LCSC (none) -> C15742
Changed lines of the file:
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@@
+			)
+		)
+		(property "LCSC" "C15742 "
+			(at 182.88 144.78 0)
+			(effects
+				(font
+					(size 1.27 1.27)
+				)
+				(hide yes)
 			)
 		)
