File: hardware/icarus/icarus.kicad_pcb (KiCad board)
At the start: 4 copper layers, 37.1 x 43.3 mm, 43 parts, among them J1 BAT, J2 IO, J3 I2C_EX, J4 UART, P1 USB_C_Plug_USB2.0, Q1 DMG2305, SW1 USER, SW2 RST, U1 AMS1117-3.3, U2 BMM150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

Commit message: Update actions
Parts:
- removed the G*** at (149.1, 52.6)
- removed J4: UART, Connector_PinHeader_2.54mm:PinHeader_1x02_P2.54mm_Vertical
- removed R13: 10k, Resistor_SMD:R_0402_1005Metric
- removed U7: ESP32-C3-MINI-1, Espressif:ESP32-C3-MINI-1
- added C10: 100nF, Capacitor_SMD:C_0402_1005Metric, F.Cu at (157.2, 60.5)
- added C11: 20pF, Capacitor_SMD:C_0402_1005Metric, F.Cu at (151.0, 66.0)
- added C12: 2.2uF, Capacitor_SMD:C_0402_1005Metric, F.Cu at (158.2, 54.2)
- added C13: 2.2uF, Capacitor_SMD:C_0402_1005Metric, F.Cu at (144.5, 51.2)
- added C14: 100nF, Capacitor_SMD:C_0402_1005Metric, F.Cu at (141.8, 59.8)
- added C15: 100nF, Capacitor_SMD:C_0402_1005Metric, F.Cu at (152.2, 66.0)
- added C16: 4.7uF, Capacitor_SMD:C_0402_1005Metric, F.Cu at (158.2, 51.8)
- added C17: 100nF, Capacitor_SMD:C_0402_1005Metric, F.Cu at (158.2, 53.0)
- added C6: 20pF, Capacitor_SMD:C_0402_1005Metric, F.Cu at (145.2, 66.0)
- added C9: 100nF, Capacitor_SMD:C_0402_1005Metric, F.Cu at (141.8, 61.0)
- added R7: 100, Resistor_SMD:R_0402_1005Metric, F.Cu at (141.8, 80.2)
- added U3: STM32F405RGTx, Package_QFP:LQFP-64_10x10mm_P0.5mm, F.Cu at (149.8, 57.3)
- added Y1: 12MHz, Crystal:Crystal_SMD_3225-4Pin_3.2x2.5mm, F.Cu at (148.1, 65.9)
- J3: value I2C_EX -> swd; footprint Connector_PinHeader_2.54mm:PinHeader_1x02_P2.54mm_Vertical -> Connector_PinHeader_1.00mm:PinHeader_1x02_P1.00mm_Vertical
- SW1: value USER -> BOOT
- moved J3 46.5 mm to (137.0, 90.0), turned to -90 degrees
- moved R3 16.9 mm to (154.7, 69.8), turned to 0 degrees
- moved J2 14.3 mm to (132.8, 77.7), turned to 180 degrees
- moved R2 9.18 mm to (154.7, 68.8)
- moved U6 4.63 mm to (141.5, 67.1)
- moved C7 4.63 mm to (140.9, 69.3)
- moved C8 4.63 mm to (142.0, 69.3)
- moved D4 2.81 mm to (141.9, 75.8)
- moved G*** 0.59 mm to (136.8, 52.8)
Connections:
- J2 pad 1: /io1 -> /pwm1
- J2 pad 2: /io2 -> /pwm2
- J2 pad 3: /io3 -> /pwm3
- J2 pad 4: /io4 -> /pwm4
- J2 pad 5: /io5 -> /usart_tx
- J2 pad 6: /io6 -> /usart_rx
- J3 pad 1: /sda -> /swdio
- J3 pad 2: /scl -> /swclk
- R12 pad 1: +3V3 -> /boot0
- R12 pad 2: /user_btn -> GND
- SW1 pad 1: GND -> /boot0
- SW1 pad 2: /user_btn -> +3V3
Routing:
- net Net-(J4-Pad2): track 104.9 -> 0.00 mm
- net Net-(J4-Pad1): track 75.9 -> 0.00 mm
- net /swdio: track 0.00 -> 63.8 mm
- net /boot0: track 0.00 -> 54.3 mm
- net /swclk: track 0.00 -> 53.5 mm
- net /nreset: track 80.0 -> 28.8 mm
- net /stat: track 0.00 -> 40.8 mm, vias 0 -> 2
- net /user_btn: track 36.8 -> 0.00 mm
- net /usart_tx: track 0.00 -> 33.2 mm, vias 0 -> 2
- net /pwm1: track 0.00 -> 30.7 mm
- net /sda: track 59.0 -> 28.7 mm, vias 8 -> 4
- net /usart_rx: track 0.00 -> 29.6 mm, vias 0 -> 2
- net /pwm2: track 0.00 -> 29.3 mm
- net /pwm3: track 0.00 -> 27.6 mm
- net /pwm4: track 0.00 -> 26.9 mm, vias 0 -> 2
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- added copper zone on F.Cu, net GND
- removed copper zone on F.Cu, net (none)
Other:
- board text added: "icarus :: Rev E nnarain"
- board text removed: "1"
- board text removed: "2"
- board text removed: "4"
- board text removed: "6"
- board text removed: "RX"
- board text removed: "SCL"
- board text removed: "SDA"
- board text removed: "TX"
- board text removed: "icarus :: Rev D.2 nnarain"
